File: 5v-boost-regulator/5v-boost-regulator.kicad_sch (KiCad schematic)
At the start: 11 parts, among them J1 Conn_01x02, U1 TPS61032PWPR

Commit message: update
Parts:
- L1: footprint (none) -> Inductor_SMD:L_Sunlord_MWSA1004S
Changed lines of the file:
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@@
 			)
 		)
-		(property "Footprint" ""
+		(property "Footprint" "Inductor_SMD:L_Sunlord_MWSA1004S"
 			(at 76.2 52.07 0)
 			(effects
