File: 5v-boost-regulator/5v-boost-regulator.kicad_sch (KiCad schematic)
At the start: 11 parts, among them J1 Conn_01x02, U1 TPS61032PWPR

Commit message: update
Parts:
- C2: value C -> 2.2uF
- C3: value C_Polarized -> 220uF; footprint (none) -> Capacitor_SMD:CP_Elec_6.3x7.7; LCSC (none) -> C2887273
- L1: LCSC (none) -> C2921230
Changed lines of the file:
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@@
 			)
 		)
-		(property "Value" "C_Polarized"
+		(property "Value" "220uF"
 			(at 195.58 61.3409 0)
 			(effects
@@
 			)
 		)
-		(property "Footprint" ""
+		(property "Footprint" "Capacitor_SMD:CP_Elec_6.3x7.7"
 			(at 192.7352 64.77 0)
 			(effects
@@
 		)
 		(property "Description" "Polarized capacitor"
+			(at 191.77 60.96 0)
+			(effects
+				(font
+					(size 1.27 1.27)
+				)
+				(hide yes)
+			)
+		)
+		(property "LCSC" "C2887273"
 			(at 191.77 60.96 0)
 			(effects
@@
 			)
 		)
+		(property "LCSC" "C2921230"
+			(at 76.2 52.07 90)
+			(effects
+				(font
+					(size 1.27 1.27)
+				)
+				(hide yes)
+			)
+		)
 		(pin "2"
 		)
@@
 			)
 		)
-		(property "Value" "C"
+		(property "Value" "2.2uF"
 			(at 184.15 62.2299 0)
 			(effects

Commit message: update
Parts:
- R1: value R -> 1M95
- R2: value R -> 390k
- R3: value R -> 1M62
- R4: value R -> 180k
Changed lines of the file:
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@@
 			)
 		)
-		(property "Value" "R"
+		(property "Value" "180k"
 			(at 171.45 69.8499 0)
 			(effects
@@
 			)
 		)
-		(property "Value" "R"
+		(property "Value" "1M62"
 			(at 171.45 62.2299 0)
 			(effects
@@
 			)
 		)
-		(property "Value" "R"
+		(property "Value" "1M95"
 			(at 85.09 69.8499 0)
 			(effects
@@
 			)
 		)
-		(property "Value" "R"
+		(property "Value" "390k"
 			(at 85.09 77.4699 0)
 			(effects

Commit message: update
Parts:
- added J2: Conn_01x02, Connector_PinHeader_2.54mm:PinHeader_1x02_P2.54mm_Horizontal, symbol Connector_Generic:Conn_01x02
Connections:
- net +5V: now also J2.1 (Pin_1)
- net at R5.2, U1.10 (LBO): now also J2.2 (Pin_2)
Changed lines of the file:
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@@
+	)
+	(junction
+		(at 207.01 81.28)
+		(diameter 0)
+		(color 0 0 0 0)
 	)
 	(junction
@@
 	(wire
 		(pts
+			(xy 207.01 81.28) (xy 222.25 81.28)
+		)
+		(stroke
+			(width 0)
+			(type default)
+		)
+	)
+	(wire
+		(pts
 			(xy 162.56 67.31) (xy 162.56 81.28)
 		)
@@
 	(wire
 		(pts
+			(xy 222.25 69.85) (xy 222.25 57.15)
+		)
+		(stroke
+			(width 0)
+			(type default)
+		)
+	)
+	(wire
+		(pts
 			(xy 154.94 54.61) (xy 154.94 57.15)
 		)
@@
 	(wire
 		(pts
+			(xy 222.25 57.15) (xy 207.01 57.15)
+		)
+		(stroke
+			(width 0)
+			(type default)
+		)
+	)
+	(wire
+		(pts
 			(xy 82.55 64.77) (xy 111.76 64.77)
 		)
@@
 		(pts
 			(xy 207.01 81.28) (xy 207.01 76.2)
+		)
+		(stroke
+			(width 0)
+			(type default)
+		)
+	)
+	(wire
+		(pts
+			(xy 222.25 72.39) (xy 222.25 81.28)
 		)
 		(stroke
@@
 					(unit 1)
 				)
+			)
+		)
+	)
+	(symbol
+		(lib_id "Connector_Generic:Conn_01x02")
+		(at 227.33 69.85 0)
+		(unit 1)
+		(exclude_from_sim no)
+		(in_bom yes)
+		(on_board yes)
+		(dnp no)
+		(fields_autoplaced yes)
+		(property "Reference" "J2"
+			(at 229.87 69.8499 0)
+			(effects
+				(font
+					(size 1.27 1.27)
+				)
+				(justify left)
+			)
+		)
+		(property "Value" "Conn_01x02"
+			(at 229.87 72.3899 0)
+			(effects
+				(font
+					(size 1.27 1.27)
+				)
+				(justify left)
+			)
+		)
+		(property "Footprint" "Connector_PinHeader_2.54mm:PinHeader_1x02_P2.54mm_Horizontal"
+			(at 227.33 69.85 0)
+			(effects
+				(font
+					(size 1.27 1.27)
+				)
+				(hide yes)
+			)
+		)
+		(property "Datasheet" "~"
+			(at 227.33 69.85 0)
+			(effects
+				(font
+					(size 1.27 1.27)
+				)
+				(hide yes)
+			)
+		)
+		(property "Description" "Generic connector, single row, 01x02, script generated (kicad-library-utils/schlib/autogen/connector/)"
+			(at 227.33 69.85 0)
+			(effects
+				(font
+					(size 1.27 1.27)
+				)
+				(hide yes)
+			)
+		)
+		(pin "1"
+		)
+		(pin "2"
+		)
+		(instances
+			(project "5v-boost-regulator"
+				(path "/0c6e4b34-a633-48f7-bd69-b032874f9ac7"
+					(reference "J2")
+					(unit 1)
+				)
