File: 5v-boost-regulator/5v-boost-regulator.kicad_pcb (KiCad board)
At the start: 2 copper layers, 49 x 25 mm, 12 parts, among them J1 Conn_01x02, J2 Conn_01x02, U1 TPS61032PWPR

Commit message: update
Routing:
- net VBat: track 55.9 -> 63.5 mm
- net Net-(L1-Pad1): track 19.0 -> 21.5 mm
- net GND: vias 0 -> 9
- added copper zone on B.Cu, net GND
- added copper zone on F.Cu, net GND
Changed lines of the file:
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@@
+	)
+	(segment
+		(start 127.2 81.8)
+		(end 127.75 81.25)
+		(width 0.4)
+		(layer "F.Cu")
+		(net 1)
 	)
 	(segment
@@
 	)
 	(segment
+		(start 127.2 81.87)
+		(end 127.2 81.8)
+		(width 0.4)
+		(layer "F.Cu")
+		(net 1)
+	)
+	(segment
 		(start 105 69.5)
 		(end 106 68.5)
@@
 	)
 	(segment
-		(start 127.2 81.87)
-		(end 133.85995 81.87)
-		(width 0.4)
-		(layer "F.Cu")
-		(net 1)
-	)
-	(segment
-		(start 134.7 83.3)
-		(end 134.26 83.74)
+		(start 128.37 81.87)
+		(end 127.75 81.25)
 		(width 0.4)
 		(layer "F.Cu")
@@
 	)
 	(segment
-		(start 126.63 82.44)
-		(end 127.2 81.87)
+		(start 127.2 81.87)
+		(end 126.63 82.44)
 		(width 0.4)
 		(layer "F.Cu")
@@
 	)
 	(segment
+		(start 133.85995 81.87)
+		(end 128.5 81.87)
+		(width 0.4)
+		(layer "F.Cu")
+		(net 1)
+	)
+	(segment
 		(start 112 71)
 		(end 114.5 68.5)
@@
 	)
 	(segment
+		(start 132.37 83.74)
+		(end 134.26 83.74)
+		(width 0.4)
+		(layer "F.Cu")
+		(net 1)
+	)
+	(segment
 		(start 134.7 82.71005)
+		(end 133.85995 81.87)
+		(width 0.4)
+		(layer "F.Cu")
+		(net 1)
+	)
+	(segment
+		(start 134.26 83.74)
 		(end 134.7 83.3)
 		(width 0.4)
@@
 	)
 	(segment
-		(start 134.26 83.74)
-		(end 132.37 83.74)
-		(width 0.4)
-		(layer "F.Cu")
-		(net 1)
-	)
-	(segment
-		(start 133.85995 81.87)
+		(start 127.75 75.5)
+		(end 127.75 81.25)
+		(width 1.2)
+		(layer "F.Cu")
+		(net 1)
+	)
+	(segment
+		(start 134.7 83.3)
 		(end 134.7 82.71005)
 		(width 0.4)
@@
 	)
 	(segment
+		(start 128.5 81.87)
+		(end 128.37 81.87)
+		(width 0.4)
+		(layer "F.Cu")
+		(net 1)
+	)
+	(segment
+		(start 128.5 81.87)
+		(end 127.2 81.87)
+		(width 0.4)
+		(layer "F.Cu")
+		(net 1)
+	)
+	(segment
 		(start 106 68.5)
 		(end 115 68.5)
@@
 		(layer "F.Cu")
 		(net 1)
+	)
+	(via
+		(at 130.25 86)
+		(size 0.4)
+		(drill 0.2)
+		(layers "F.Cu" "B.Cu")
+		(net 2)
+	)
+	(via
+		(at 128.5 83.5)
+		(size 0.4)
+		(drill 0.2)
+		(layers "F.Cu" "B.Cu")
+		(net 2)
+	)
+	(via
+		(at 126.75 83.75)
+		(size 0.4)
+		(drill 0.2)
+		(layers "F.Cu" "B.Cu")
+		(net 2)
+	)
+	(via
+		(at 128.75 86)
+		(size 0.4)
+		(drill 0.2)
+		(layers "F.Cu" "B.Cu")
+		(net 2)
+	)
+	(via
+		(at 126.25 83.75)
+		(size 0.4)
+		(drill 0.2)
+		(layers "F.Cu" "B.Cu")
+		(net 2)
+	)
+	(via
+		(at 132.75 85.75)
+		(size 0.4)
+		(drill 0.2)
+		(layers "F.Cu" "B.Cu")
+		(net 2)
+	)
+	(via
+		(at 127.25 83.75)
+		(size 0.4)
+		(drill 0.2)
+		(layers "F.Cu" "B.Cu")
+		(net 2)
+	)
+	(via
+		(at 132 85.75)
+		(size 0.4)
+		(drill 0.2)
+		(layers "F.Cu" "B.Cu")
+		(net 2)
+	)
+	(via
+		(at 130.25 83.5)
+		(size 0.4)
+		(drill 0.2)
+		(layers "F.Cu" "B.Cu")
+		(net 2)
 	)
 	(segment
@@
 	)
 	(segment
+		(start 132.37 86.35)
+		(end 133.35 86.35)
+		(width 0.4)
+		(layer "F.Cu")
+		(net 4)
+	)
+	(segment
 		(start 137.25 82.75)
 		(end 137.25 75.5)
@@
 	)
 	(segment
+		(start 132.37 87)
+		(end 134 87)
+		(width 1.2)
+		(layer "F.Cu")
+		(net 4)
+	)
+	(segment
 		(start 139.5 86)
 		(end 139.5 85)
@@
 	)
 	(segment
-		(start 132.37 87)
+		(start 134 87)
 		(end 138.5 87)
 		(width 1.2)
+		(layer "F.Cu")
+		(net 4)
+	)
+	(segment
+		(start 133.35 86.35)
+		(end 134 87)
+		(width 0.4)
+		(layer "F.Cu")
+		(net 4)
+	)
+	(segment
+		(start 132.37 86.35)
+		(end 132.37 87)
+		(width 0.4)
 		(layer "F.Cu")
 		(net 4)
@@
 		(net 8)
 	)
+	(zone
+		(net 2)
+		(net_name "GND")
+		(layers "F&B.Cu")
+		(hatch edge 0.5)
+		(connect_pads
+			(clearance 0.5)
+		)
+		(min_thickness 0.25)
+		(filled_areas_thickness no)
+		(fill yes
+			(thermal_gap 0.5)
+			(thermal_bridge_width 0.5)
+		)
+		(polygon
+			(pts
+				(xy 99 67.5) (xy 148 67.5) (xy 148 92.5) (xy 99 92.5)
+			)
+		)
+	)
 )
